Commit message: Separate robot spawn to individual files
Signed-off-by: Camilo Andres Alvis Bautista <kmilo7204@gmail.com>

File: Project-3/catkin_ws/src/diff_robot/urdf/diff_robot.xacro (robot description, xacro)
@@ -1,12 +1,18 @@
 <robot name="diff_robot" xmlns:xacro="http://www.ros.org/wiki/xacro">
-  <xacro:include filename="$(find diff_robot)/urdf/diff_robot.gazebo" />
+  <xacro:include filename="$(find diff_robot)/urdf/diff_robot.gazebo"/>
+  <xacro:property name="x" default="0.0"/>
+  <xacro:property name="y" default="0.0"/>
+  <xacro:property name="z" default="0.0"/>
+  <xacro:property name="roll" default="0.0"/>
+  <xacro:property name="pitch" default="0.0"/>
+  <xacro:property name="yaw" default="0.0"/>
   <link name="robot_footprint"></link>
   <joint name="robot_footprint_joint" type="fixed">
-    <origin xyz="0 0 0" rpy="0 0 0" />
+    <origin xyz="${x} ${y} ${z}" rpy="${roll} ${pitch} ${yaw}"/>
     <parent link="robot_footprint"/>
     <child link="chassis" />
   </joint>
   <link name='chassis'>
-    <pose>0 0 0.1 0 0 0</pose>
+    <pose>5 0 0.1 0 0 0</pose>
     <inertial>
       <mass value="15.0"/>
