Commit message: Add RGB sensor and documentaiton
Signed-off-by: Camilo Andres Alvis Bautista <kmilo7204@gmail.com>

File: Project-4/catkin_ws/src/diff_robot/urdf/diff_robot.xacro (robot description, xacro)
@@ -130,4 +130,6 @@
     </inertial>
   </link>
+  <link name="camera_link_optical">
+  </link>
   <!-- Laser scan -->
   <link name="hokuyo">
@@ -181,3 +183,8 @@
     <axis xyz="0 1 0" rpy="0 0 0"/>
   </joint>
+  <joint name="camera_optical_joint" type="fixed">
+    <origin xyz="0 0 0" rpy="-1.5707 0 -1.5707"/>
+    <parent link="camera"/>
+    <child link="camera_link_optical"/>
+  </joint>
 </robot>
